File: 3_Flight_Computer/PCB/ALBERT_FLIGHTCOMPUTER/Sensors.kicad_sch (KiCad schematic)
At the start: 20 parts, among them IC1 BMP390, U1 ZOE-M8Q, U3 BMI088, U4 LSM6DSLTR, U5 BMM150, Y3 CM7V-T1A-32.768KHZ-6PF-20PPM-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

Commit message: Add lock file for ALBERT_FLIGHTCOMPUTER PCB design
Parts:
- removed C50: 100n, symbol Device:C
- removed C51: 4u7, symbol Device:C
- removed L3: 2u2, symbol Device:L
- removed U1: ZOE-M8Q, RF_GPS:ublox_ZOE_M8, symbol RF_GPS:ZOE-M8Q
- removed Y3: CM7V-T1A-32.768KHZ-6PF-20PPM-TA-QC, CM7V32768TBQA020, symbol CM7V-T1A-32_768KHZ-6PF-20PPM-T:CM7V-T1A-32.768KHZ-6PF-20PPM-TA-QC
- C33: renamed from C18; footprint (none) -> Capacitor_SMD:C_0402_1005Metric
- C34: renamed from C47; footprint (none) -> Capacitor_SMD:C_0402_1005Metric
- C35: renamed from C17; footprint (none) -> Capacitor_SMD:C_0402_1005Metric
- C36: renamed from C48; footprint (none) -> Capacitor_SMD:C_0402_1005Metric
- C37: renamed from C46; footprint (none) -> Capacitor_SMD:C_0402_1005Metric
- C38: renamed from C15; footprint (none) -> Capacitor_SMD:C_0402_1005Metric
- C39: renamed from C45; footprint (none) -> Capacitor_SMD:C_0402_1005Metric
- C40: renamed from C16; footprint (none) -> Capacitor_SMD:C_0402_1005Metric
- IC3: renamed from IC1; footprint BMP390 -> BMP390:BMP390
- R35: renamed from R5; footprint (none) -> Resistor_SMD:R_0402_1005Metric
- R36: renamed from R3; footprint (none) -> Resistor_SMD:R_0402_1005Metric
- R37: renamed from R4; footprint (none) -> Resistor_SMD:R_0402_1005Metric
- renumbered U4 to U1, U3 to U2, U5 to U3
Connections:
- net SPI1_IMU1_CSB_ACCEL renamed SPI1_CS_ACCEL_NAV
- net SPI1_IMU1_CSB_GYRO renamed SPI1_CS_GYRO_NAV
- net SPI1_IMU1_INT_ACCEL renamed SPI1_INT_ACCEL_NAV
- net SPI1_IMU1_INT_GYRO renamed SPI1_INT_GYRO_NAV
- net SPI1_IMU1_MISO renamed SPI1_MISO_NAV
- net SPI1_IMU1_MOSI renamed SPI1_MOSI_NAV
- net SPI1_IMU1_SCK renamed SPI1_SCK_NAV
- net SPI2_BAR_CSB renamed SPI2_CS_NAV
- net SPI2_BAR_INT renamed SPI2_INT_NAV
- net SPI2_BAR_MISO renamed SPI2_MISO_NAV
- net SPI2_BAR_MOSI renamed SPI2_MOSI_NAV
- net SPI2_BAR_SCK renamed SPI2_SCK_NAV
- no-connect marks 5 -> 6
Other:
- company: (none) -> ALBERT AEROSPACE
- moved on the sheet: C33, C34, C35, C36, C37, C38, C39, C40, IC3, R35, R36, R37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

Commit message: Add production files and update project lock file
- Added new production IT1 zip file for ALBERT_FLIGHTCOMPUTER.
- Removed obsolete test zip file from production directory.
- Created a lock file for the KiCad schematic with user and hostname information.
Parts:
- C33, C34, C35, C36, C37, C38, C39, C40: LCSC (none) -> C1525
- IC3: LCSC (none) -> C5124834
- R35, R36, R37: LCSC (none) -> C25796
- U1: LCSC (none) -> C126672
- U2: LCSC (none) -> C194919
- U3: LCSC (none) -> C171681
