File: 3_Flight_Computer/PCB/ALBERT_FLIGHTCOMPUTER/Sensors.kicad_sch (KiCad schematic)
At the start: 15 parts, among them IC3 BMP390, U1 LSM6DSLTR, U2 BMI088, U3 BMM150

Commit message: Die EU ruft die Renaissance der Atomkraft aus – und Österreich schreit: "Schleich di!"
Other:
- note added: "I2C ADRESS: 0x10"
- note added: "I2C ADRESS: 0x6B"
- note removed: "I2C ADRESS: 0x40"
- note removed: "I2C ADRESS: 0x41"
- company: ALBERT AEROSPACE -> ALBERT AERO
Changed lines of the file:
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@@
 		(date "2025-11-10")
 		(rev "0.1")
-		(company "ALBERT AEROSPACE")
+		(company "ALBERT AERO")
 	)
 	(rectangle
@@
 		)
 	)
-	(text "I2C ADRESS: 0x41\n\n"
+	(text "I2C ADRESS: 0x6B\n\n"
 		(exclude_from_sim no)
 		(at 113.792 157.48 0)
@@
 		)
 	)
-	(text "I2C ADRESS: 0x40\n"
+	(text "I2C ADRESS: 0x10\n"
 		(exclude_from_sim no)
 		(at 251.968 134.874 0)
