File: 3_Flight_Computer/PCB/ALBERT_FLIGHTCOMPUTER/_autosave-Sensors.kicad_sch (KiCad schematic)
At the start: 20 parts, among them IC1 BMP390, U1 ZOE-M8Q, U3 BMI088, U4 LSM6DSLTR, U5 BMM150, Y3 CM7V-T1A-32.768KHZ-6PF-20PPM-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

Commit message: Refactor code structure for improved readability and maintainability
Connections:
- net GND: now also U1.C1 (SQI_D1), U1.D3 (~{SQI_CS}), U1.E1 (SQI_CLK), U1.E3 (SQI_D2), U1.F3 (SQI_D3)
Other:
- moved on the sheet: C50, C51, L3
Changed lines of the file:
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@@
 	)
 	(junction
+		(at 52.07 123.19)
+		(diameter 0)
+		(color 0 0 0 0)
+	)
+	(junction
 		(at 130.81 50.8)
 		(diameter 0)
@@
 	)
 	(junction
+		(at 52.07 128.27)
+		(diameter 0)
+		(color 0 0 0 0)
+	)
+	(junction
 		(at 222.25 85.09)
 		(diameter 0)
@@
 	)
 	(junction
-		(at 128.27 127)
+		(at 114.3 127)
 		(diameter 0)
 		(color 0 0 0 0)
@@
 	)
 	(junction
-		(at 128.27 191.77)
+		(at 114.3 191.77)
 		(diameter 0)
 		(color 0 0 0 0)
@@
 	)
 	(junction
+		(at 52.07 125.73)
+		(diameter 0)
+		(color 0 0 0 0)
+	)
+	(junction
 		(at 222.25 87.63)
 		(diameter 0)
@@
 	)
 	(junction
+		(at 52.07 130.81)
+		(diameter 0)
+		(color 0 0 0 0)
+	)
+	(junction
 		(at 201.93 129.54)
 		(diameter 0)
@@
 	(wire
 		(pts
-			(xy 78.74 191.77) (xy 128.27 191.77)
+			(xy 78.74 191.77) (xy 114.3 191.77)
 		)
 		(stroke
@@
 	(wire
 		(pts
-			(xy 147.32 106.68) (xy 147.32 140.97)
+			(xy 52.07 130.81) (xy 55.88 130.81)
+		)
+		(stroke
+			(width 0)
+			(type default)
+		)
+	)
+	(wire
+		(pts
+			(xy 133.35 106.68) (xy 133.35 140.97)
 		)
 		(stroke
@@
 	(wire
 		(pts
-			(xy 121.92 111.76) (xy 121.92 127)
+			(xy 107.95 111.76) (xy 107.95 127)
 		)
 		(stroke
@@
 	(wire
 		(pts
+			(xy 55.88 120.65) (xy 52.07 120.65)
+		)
+		(stroke
+			(width 0)
+			(type default)
+		)
+	)
+	(wire
+		(pts
 			(xy 163.83 85.09) (xy 163.83 80.01)
 		)
@@
 	(wire
 		(pts
+			(xy 52.07 123.19) (xy 52.07 125.73)
+		)
+		(stroke
+			(width 0)
+			(type default)
+		)
+	)
+	(wire
+		(pts
 			(xy 217.17 85.09) (xy 222.25 85.09)
 		)
@@
 	(wire
 		(pts
+			(xy 52.07 128.27) (xy 52.07 130.81)
+		)
+		(stroke
+			(width 0)
+			(type default)
+		)
+	)
+	(wire
+		(pts
 			(xy 222.25 87.63) (xy 234.95 87.63)
 		)
@@
 	(wire
 		(pts
-			(xy 147.32 148.59) (xy 147.32 191.77)
+			(xy 133.35 148.59) (xy 133.35 191.77)
 		)
 		(stroke
@@
 	(wire
 		(pts
-			(xy 121.92 127) (xy 128.27 127)
+			(xy 107.95 127) (xy 114.3 127)
 		)
 		(stroke
@@
 	(wire
 		(pts
-			(xy 128.27 110.49) (xy 128.27 114.3)
+			(xy 52.07 125.73) (xy 52.07 128.27)
+		)
+		(stroke
+			(width 0)
+			(type default)
+		)
+	)
+	(wire
+		(pts
+			(xy 114.3 110.49) (xy 114.3 114.3)
 		)
 		(stroke
@@
 	(wire
 		(pts
-			(xy 128.27 148.59) (xy 128.27 191.77)
+			(xy 114.3 148.59) (xy 114.3 191.77)
 		)
 		(stroke
@@
 	(wire
 		(pts
+			(xy 52.07 125.73) (xy 55.88 125.73)
+		)
+		(stroke
+			(width 0)
+			(type default)
+		)
+	)
+	(wire
+		(pts
 			(xy 80.01 58.42) (xy 80.01 73.66)
 		)
@@
 	(wire
 		(pts
-			(xy 71.12 106.68) (xy 147.32 106.68)
+			(xy 71.12 106.68) (xy 133.35 106.68)
 		)
 		(stroke
@@
 	(wire
 		(pts
-			(xy 128.27 127) (xy 128.27 140.97)
+			(xy 114.3 127) (xy 114.3 140.97)
 		)
 		(stroke
@@
 	(wire
 		(pts
-			(xy 81.28 110.49) (xy 128.27 110.49)
+			(xy 81.28 110.49) (xy 114.3 110.49)
 		)
 		(stroke
@@
 	(wire
 		(pts
+			(xy 52.07 120.65) (xy 52.07 123.19)
+		)
+		(stroke
+			(width 0)
+			(type default)
+		)
+	)
+	(wire
+		(pts
 			(xy 179.07 100.33) (xy 179.07 105.41)
 		)
@@
 	(wire
 		(pts
-			(xy 128.27 121.92) (xy 128.27 127)
+			(xy 114.3 121.92) (xy 114.3 127)
 		)
 		(stroke
@@
 	(wire
 		(pts
+			(xy 52.07 123.19) (xy 55.88 123.19)
+		)
+		(stroke
+			(width 0)
+			(type default)
+		)
+	)
+	(wire
+		(pts
 			(xy 80.01 55.88) (xy 80.01 58.42)
 		)
@@
 	(wire
 		(pts
+			(xy 52.07 128.27) (xy 55.88 128.27)
+		)
+		(stroke
+			(width 0)
+			(type default)
+		)
+	)
+	(wire
+		(pts
 			(xy 124.46 40.64) (xy 124.46 39.37)
 		)
@@
 	(wire
 		(pts
-			(xy 86.36 111.76) (xy 121.92 111.76)
+			(xy 86.36 111.76) (xy 107.95 111.76)
 		)
 		(stroke
@@
 	(wire
 		(pts
-			(xy 128.27 191.77) (xy 147.32 191.77)
+			(xy 114.3 191.77) (xy 133.35 191.77)
 		)
 		(stroke
@@
 	)
 	(symbol
+		(lib_id "power:GND")
+		(at 52.07 130.81 0)
+		(unit 1)
+		(exclude_from_sim no)
+		(in_bom yes)
+		(on_board yes)
+		(dnp no)
+		(fields_autoplaced yes)
+		(property "Reference" "#PWR0104"
+			(at 52.07 137.16 0)
+			(effects
+				(font
+					(size 1.27 1.27)
+				)
+				(hide yes)
+			)
+		)
+		(property "Value" "GND"
+			(at 52.07 135.89 0)
+			(effects
+				(font
+					(size 1.27 1.27)
+				)
+				(hide yes)
+			)
+		)
+		(property "Footprint" ""
+			(at 52.07 130.81 0)
+			(effects
+				(font
+					(size 1.27 1.27)
+				)
+				(hide yes)
+			)
+		)
+		(property "Datasheet" ""
+			(at 52.07 130.81 0)
+			(effects
+				(font
+					(size 1.27 1.27)
+				)
+				(hide yes)
+			)
+		)
+		(property "Description" "Power symbol creates a global label with name \"GND\" , ground"
+			(at 52.07 130.81 0)
+			(effects
+				(font
+					(size 1.27 1.27)
+				)
+				(hide yes)
+			)
+		)
+		(pin "1"
+		)
+		(instances
+			(project "ALBERT_FLIGHTCOMPUTER"
+				(path "/caf1b85f-a91d-4c85-9df1-65f9ebc85027/f7ea2c19-61e9-4cc6-adc7-384d26cb19eb"
+					(reference "#PWR0104")
+					(unit 1)
+				)
+			)
+		)
+	)
+	(symbol
 		(lib_id "Device:C")
 		(at 224.79 143.51 0)
@@
 	(symbol
 		(lib_id "Device:C")
-		(at 128.27 144.78 0)
+		(at 114.3 144.78 0)
 		(unit 1)
 		(exclude_from_sim no)
@@
 		(fields_autoplaced yes)
 		(property "Reference" "C51"
-			(at 132.08 143.5099 0)
+			(at 118.11 143.5099 0)
 			(effects
 				(font
@@
 		)
 		(property "Value" "4u7"
-			(at 132.08 146.0499 0)
+			(at 118.11 146.0499 0)
 			(effects
 				(font
@@
 		)
 		(property "Footprint" ""
-			(at 129.2352 148.59 0)
+			(at 115.2652 148.59 0)
 			(effects
 				(font
@@
 		)
 		(property "Datasheet" "~"
-			(at 128.27 144.78 0)
+			(at 114.3 144.78 0)
 			(effects
 				(font
@@
 		)
 		(property "Description" "Unpolarized capacitor"
-			(at 128.27 144.78 0)
+			(at 114.3 144.78 0)
 			(effects
 				(font
@@
 	(symbol
 		(lib_id "Device:L")
-		(at 128.27 118.11 0)
+		(at 114.3 118.11 0)
 		(unit 1)
 		(exclude_from_sim no)
@@
 		(fields_autoplaced yes)
 		(property "Reference" "L3"
-			(at 129.54 116.8399 0)
+			(at 115.57 116.8399 0)
 			(effects
 				(font
@@
 		)
 		(property "Value" "2u2"
-			(at 129.54 119.3799 0)
+			(at 115.57 119.3799 0)
 			(effects
 				(font
@@
 		)
 		(property "Footprint" ""
-			(at 128.27 118.11 0)
+			(at 114.3 118.11 0)
 			(effects
 				(font
@@
 		)
 		(property "Datasheet" "~"
-			(at 128.27 118.11 0)
+			(at 114.3 118.11 0)
 			(effects
 				(font
@@
 		)
 		(property "Description" "Inductor"
-			(at 128.27 118.11 0)
+			(at 114.3 118.11 0)
 			(effects
 				(font
@@
 	(symbol
 		(lib_id "Device:C")
-		(at 147.32 144.78 0)
+		(at 133.35 144.78 0)
 		(unit 1)
 		(exclude_from_sim no)
@@
 		(fields_autoplaced yes)
 		(property "Reference" "C50"
-			(at 151.13 143.5099 0)
+			(at 137.16 143.5099 0)
 			(effects
 				(font
@@
 		)
 		(property "Value" "100n"
-			(at 151.13 146.0499 0)
+			(at 137.16 146.0499 0)
 			(effects
 				(font
@@
 		)
 		(property "Footprint" ""
-			(at 148.2852 148.59 0)
+			(at 134.3152 148.59 0)
 			(effects
 				(font
@@
 		)
 		(property "Datasheet" "~"
-			(at 147.32 144.78 0)
+			(at 133.35 144.78 0)
 			(effects
 				(font
@@
 		)
 		(property "Description" "Unpolarized capacitor"
-			(at 147.32 144.78 0)
+			(at 133.35 144.78 0)
 			(effects
 				(font
