File: 3_Flight_Computer/PCB/ALBERT_FLIGHTCOMPUTER/ALBERT_FLIGHTCOMPUTER.kicad_pcb (KiCad board)
At the start: 4 copper layers, 73 x 98 mm, 159 parts, among them IC1 PCA9685PW,118, IC2 W25N01GVZEIG, IC3 BMP390, J1 Conn_01x05, J10 Conn_01x06, J11 USB_C_Receptacle_USB2.0_14P, J12 Conn_02x08_Odd_Even, J15 Conn_01x08, J16 Conn_01x05, J17 XT60-M, J18 5-1814400-2, J19 5-1814400-2, J2 USB_C_Receptacle_USB2.0_14P, J3 Screw_Terminal_01x02, J4 Screw_Terminal_01x02, J5 Screw_Terminal_01x02, J6 Screw_Terminal_01x02, J7 Micro_SD_Card_Det2, J8 Conn_01x04, J9 Conn_01x04, Q1 BSC028N06LS3, Q2 BSC028N06LS3, Q3 BSC028N06LS3, Q4 BSC028N06LS3, SW1 SW_SPDT, SW2 SW_SPDT, U1 LSM6DSLTR, U2 BMI088, U3 BMM150, U4 AMS1117-3.3, U5 TPS54308, U6 INA219AxDCN, U7 RFM95W-868S2, U8 ZOE-M8Q, Y1 16MHz, Y2 16MHz, Y3 CM7V-T1A-32.768KHZ-6PF-20PPM-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

Commit message: update pcb
Parts:
- D7, R42: moved to F.Cu
- moved C34 7.41 mm to (111.0, 74.3), turned to 90 degrees
- moved C36 5.40 mm to (109.2, 71.5), turned to 180 degrees
- moved R19 4.83 mm to (64.8, 101.0)
- moved R16 4.63 mm to (66.2, 102.2)
- moved R20 4.63 mm to (61.9, 100.9)
- moved R21 4.63 mm to (60.6, 102.3)
- moved J7 4.63 mm to (65.0, 90.4)
- moved R11 4.45 mm to (67.9, 103.6)
- moved R15 2.62 mm to (96.9, 113.1)
- moved U1 2.17 mm to (108.4, 73.6), turned to 180 degrees
- moved C39 2.16 mm to (100.3, 79.3)
- moved C37 2.16 mm to (102.3, 77.2)
- moved U3 2.16 mm to (101.9, 79.0)
- moved R42 2.06 mm to (92.2, 92.3)
- moved FB3 1.55 mm to (93.8, 64.0)
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Connections:
- NAV1 pad 2: unconnected-(NAV1-PC13-Pad2) -> INT1_NAV
- NAV1 pad 3: unconnected-(NAV1-PC14-Pad3) -> INT2_NAV
- NAV1 pad 50: INT2_NAV -> unconnected-(NAV1-PA15-Pad50)
- NAV1 pad 51: INT1_NAV -> unconnected-(NAV1-PC10-Pad51)
Routing:
- net USART1_RX_NAV: track 0.00 -> 65.8 mm, vias 0 -> 4
- net GND: track 167.4 -> 232.8 mm, vias 98 -> 166
- net USART1_TX_NAV: track 0.00 -> 57.7 mm, vias 0 -> 2
- net NRST_MPU: track 1.76 -> 58.3 mm, vias 0 -> 2
- net INT1_NAV: track 0.00 -> 53.4 mm, vias 0 -> 2
- net +3.3V: track 90.2 -> 142.4 mm, vias 19 -> 56
- net INT2_NAV: track 0.00 -> 51.7 mm, vias 0 -> 2
- net SD_DET_MPU: track 0.00 -> 48.3 mm, vias 0 -> 3
- net GPIO2_MPU: track 0.00 -> 46.9 mm, vias 0 -> 2
- net GPIO1_MPU: track 0.00 -> 46.4 mm, vias 0 -> 1
- net GPIO5_MPU: track 0.00 -> 44.0 mm, vias 0 -> 3
- net GPIO6_MPU: track 0.00 -> 43.2 mm, vias 0 -> 3
- net GPIO3_MPU: track 0.00 -> 42.6 mm, vias 0 -> 2
- net GPIO4_MPU: track 0.00 -> 42.5 mm, vias 0 -> 2
- net SD_DAT3_MPU: track 4.10 -> 45.2 mm, vias 0 -> 1
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- added copper zone on In2.Cu, net GND
Other:
- board text added: "+"
- board text added: "-"
- board text added: "BARO"
- board text added: "DEBUG MPU"
- board text added: "DEBUG NAV"
- board text added: "FLASH"
- board text added: "GPIO MPU"
- board text added: "GPIO NAV"
- board text added: "GPS"
- board text added: "IMU1"
- board text added: "IMU2"
- board text added: "KOMADORI"
- board text added: "LDO"
- board text added: "LORA"
- board text added: "LORA MODULE"
- board text added: "MAGNETO"
- board text added: "MPU"
- board text added: "NAV"
- board text added: "PWM 0"
- board text added: "PWM 1"
- board text added: "PWM 2"
- board text added: "PWM 3"
- board text added: "PWM 4"
- board text added: "PWM 5"
- board text added: "PWM 6"
- board text added: "PWM 7"
- board text added: "Pyro 1"
- board text added: "Pyro 2"
- board text added: "Pyro 3"
- board text added: "Pyro 4"
- board text added: "SD-Card"
- board text added: "SPI"
- board text added: "UART 1"
- board text added: "UART 2"
- board text added: "USB MPU"
- board text added: "USB NAV"
- board text added: "designed by"

Commit message: Add production files and update project lock file
- Added new production IT1 zip file for ALBERT_FLIGHTCOMPUTER.
- Removed obsolete test zip file from production directory.
- Created a lock file for the KiCad schematic with user and hostname information.
Parts:
- removed HXPZ2.54-3x8PZZ1: ~, HXPZ2.54-3x8PZZ:HX PZ2.54-3x8P ZZ
- added J13: HXPZ2.54-3x8PZZ1, HXPZ2.54-3x8PZZ:HX PZ2.54-3x8P ZZ, F.Cu at (47.7, 122.7)
- added U10: USBLC6-2SC6, Package_TO_SOT_SMD:SOT-23-6, F.Cu at (82.8, 69.2)
- added U9: USBLC6-2SC6, Package_TO_SOT_SMD:SOT-23-6, F.Cu at (102.2, 109.9)
- C22, C31, C32, C5, C6, C7, C8: footprint Capacitor_Tantalum_SMD:CP_EIA-1608-10_AVX-L -> Capacitor_SMD:C_0805_2012Metric
- FB1: value 120R -> 100R
- FB2, FB3: value FerriteBead -> 100R; footprint Inductor_SMD:L_0603_1608Metric -> Inductor_SMD:L_0805_2012Metric
- FB4: value 120R -> 100R; footprint Inductor_SMD:L_0603_1608Metric -> Inductor_SMD:L_0805_2012Metric
- MPU1: value STM32H753VITx -> STM32H753VIT6
- NAV1: value STM32F405RGTx -> STM32F405RGT6
- R9: value 47 -> 22
- Y3: value CM7V-T1A-32.768KHZ-6PF-20PPM-TA-QC -> 32.768kHz; footprint CMV-T1A-32.768KHZ:CM7V32768TBQA020 -> Crystal:Crystal_SMD_MicroCrystal_CC7V-T1A-2Pin_3.2x1.5mm
- moved D5 2.95 mm to (102.3, 102.5)
- moved FB2 2.95 mm to (102.5, 98.0)
- moved C21 2.09 mm to (78.5, 69.2)
- moved C24 1.08 mm to (79.4, 70.8)
- moved R43 0.58 mm to (86.7, 68.9)
- moved C6 0.46 mm to (71.8, 125.5)
- moved C8 0.28 mm to (67.7, 119.8)
- moved C5 0.20 mm to (71.8, 123.4)
- moved C32 0.19 mm to (92.5, 87.0)
- moved FB4 0.18 mm to (91.3, 84.2)
- moved C7 0.16 mm to (75.8, 104.7)
- moved R36 0.06 mm to (101.5, 88.2)
- moved J11 0.05 mm to (82.3, 61.9)
- moved R41 0.05 mm to (76.0, 64.5)
Connections:
- J11 pad A6: USB_NAV_D+ -> /NAV/ESD_NAV_D+
- J11 pad A7: USB_NAV_D- -> /NAV/ESD_NAV_D-
- J11 pad B6: USB_NAV_D+ -> /NAV/ESD_NAV_D+
- J11 pad B7: USB_NAV_D- -> /NAV/ESD_NAV_D-
- J2 pad A6: USB_MPU_D+ -> /ESD_MPU_D+
- J2 pad A7: USB_MPU_D- -> /ESD_MPU_D-
- J2 pad B6: USB_MPU_D+ -> /ESD_MPU_D+
- J2 pad B7: USB_MPU_D- -> /ESD_MPU_D-
Routing:
- net USB_MPU_D-: track 23.4 -> 12.4 mm, vias 2 -> 0
- net USB_MPU_D+: track 23.4 -> 13.1 mm, vias 2 -> 0
- net USB_NAV_D-: track 11.5 -> 2.27 mm, vias 2 -> 0
- net USB_NAV_D+: track 11.5 -> 2.43 mm, vias 2 -> 0
- net /ESD_MPU_D+: track 0.00 -> 8.79 mm, vias 0 -> 2
- net /ESD_MPU_D-: track 0.00 -> 8.74 mm, vias 0 -> 2
- net GND: track 232.8 -> 240.7 mm, vias 166 -> 168
- net Net-(D5-A): track 13.9 -> 21.0 mm
- net /NAV/ESD_NAV_D-: track 0.00 -> 7.02 mm, vias 0 -> 2
- net /NAV/ESD_NAV_D+: track 0.00 -> 6.89 mm, vias 0 -> 2
- net Net-(D6-A): track 15.0 -> 19.5 mm
- net +5V: track 47.2 -> 48.6 mm
- net Net-(NAV1-VCAP_2): track 3.25 -> 4.58 mm
- net +3.3V: track 142.4 -> 143.7 mm
- net GPIO12_MPU: track 33.5 -> 32.5 mm
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Other:
- board text added: "KOMADORI IT0 PROJECT ALBERT 09/12/25 FELIX ZAUNER"
- board text removed: "guided by BOSCH SENSORTEC"
