File: 3_Flight_Computer/PCB/ALBERT_FLIGHTCOMPUTER/ALBERT_FLIGHTCOMPUTER.kicad_pcb (KiCad board)
At the start: 4 copper layers, 73 x 98 mm, 161 parts, among them IC1 PCA9685PW,118, IC2 W25N01GVZEIG, IC3 BMP390, J1 Conn_01x05, J10 Conn_01x06, J11 USB_C_Receptacle_USB2.0_14P, J12 Conn_02x08_Odd_Even, J13 HXPZ2.54-3x8PZZ1, J15 Conn_01x08, J16 Conn_01x05, J17 XT60-M, J18 5-1814400-2, J19 5-1814400-2, J2 USB_C_Receptacle_USB2.0_14P, J3 Screw_Terminal_01x02, J4 Screw_Terminal_01x02, J5 Screw_Terminal_01x02, J6 Screw_Terminal_01x02, J7 Micro_SD_Card_Det2, J8 Conn_01x04, J9 Conn_01x04, Q1 BSC028N06LS3, Q2 BSC028N06LS3, Q3 BSC028N06LS3, Q4 BSC028N06LS3, SW1 SW_SPDT, SW2 SW_SPDT, U1 LSM6DSLTR, U10 USBLC6-2SC6, U2 BMI088, U3 BMM150, U4 AMS1117-3.3, U5 TPS54308, U6 INA219AxDCN, U7 RFM95W-868S2, U8 ZOE-M8Q, U9 USBLC6-2SC6, Y1 16MHz, Y2 16MHz, Y3 32.768kHz

Commit message: Pregnant Women, DON’T USE TYLENOL UNLESS ABSOLUTELY NECESSARY, DON’T GIVE TYLENOL TO YOUR YOUNG CHILD FOR VIRTUALLY ANY REASON, BREAK UP THE MMR SHOT INTO THREE TOTALLY SEPARATE SHOTS (NOT MIXED!), TAKE CHICKEN P SHOT SEPARATELY, TAKE HEPATITAS B SHOT AT 12 YEARS OLD, OR OLDER, AND, IMPORTANTLY, TAKE VACCINE IN 5 SEPARATE MEDICAL VISITS! President DJT
Parts:
- added J20: Conn_01x08, Connector_PinHeader_2.54mm:PinHeader_1x08_P2.54mm_Vertical, F.Cu at (50.2, 103.9)
- J13: value HXPZ2.54-3x8PZZ1 -> Conn_02x08_Odd_Even; footprint HXPZ2.54-3x8PZZ:HX PZ2.54-3x8P ZZ -> Connector_PinHeader_2.54mm:PinHeader_2x08_P2.54mm_Vertical
- moved J13 19.0 mm to (45.0, 103.9)
Connections:
- J13 pad 10: GND -> IN-
- J13 pad 11: IN- -> GND
- J13 pad 12: PWM_03 -> IN-
- J13 pad 15: PWM_04 -> GND
- J13 pad 16: GND -> IN-
- J13 pad 3: PWM_00 -> GND
- J13 pad 4: GND -> IN-
- J13 pad 5: IN- -> GND
- J13 pad 6: PWM_01 -> IN-
- J13 pad 9: PWM_02 -> GND
