File: 3_Flight_Computer/PCB/ALBERT_FLIGHTCOMPUTER/ALBERT_FLIGHTCOMPUTER.kicad_sch (KiCad schematic)
At the start: 30 parts, among them IC1 BMP390, J1 USB_B_Micro, J2 Conn_01x04_Pin, SW1 SW_SPDT, U1 STM32F405RGTx, U2 AMS1117-3.3, U3 BMI088, U4 LSM6DSLTR, U5 BMM150, Y1 16MHz

Commit message: Refactor code structure for improved readability and maintainability
Parts:
- added C17, C18: 100n, symbol Device:C
- added R3, R4, R5: 56k, symbol Device:R
Connections:
- net +3.3V: now also IC1.1 (VDDIO), IC1.10 (VDD), C17.1, C18.1, R3.1, R4.1, R5.1
- net GND: now also IC1.3 (VSS_1), IC1.8 (VSS_2), IC1.9 (VSS_3), C17.2, C18.2
- net IMU1_INT_ACCEL: now reaches U3.16 (INT1)
- net IMU1_INT_ACCEL: no longer U3.12 (INT3)
- net IMU1_INT_GYRO: now reaches U1.24 (PC4)
- net IMU1_INT_GYRO: now also U3.12 (INT3)
- net BAR_CLK: now reaches IC1.2 (SCK)
- net BAR_MOSI: now reaches IC1.4 (SDI)
- net BAR_MISO: now reaches IC1.5 (SDO)
- net at IC1.6 (CSB): now also R5.2
- net BAR_INT: now reaches IC1.7 (INT)
- net SPI1_CSB_ACCEL renamed IMU1_CSB_ACCEL
- net IMU1_CSB_ACCEL: now also U1.11 (PC3)
- net SPI1_CSB_GYRO renamed IMU1_CSB_GYRO
- net SPI1_INTERRUPT: no longer names the net of U3.1 (INT2)
- net SPI1_INTERRUPT: no longer U1.11 (PC3)
- net SPI1_MISO renamed IMU1_MISO
- net SPI1_MOSI renamed IMU1_MOSI
- net IMU1_MOSI: now also R3.2
- net SPI1_SCK renamed IMU1_SCK
- net IMU1_SCK: now also R4.2
- no-connect marks 3 -> 4
Other:
- note added: "Pressure Sensor"
- note added: "Primary IMU"
- moved on the sheet: C15, C16, IC1, J1, J2, U3, U4, U5

Commit message: Refactor code structure for improved readability and maintainability
Parts:
- removed C13, C14: 22u, symbol Device:C
- removed C15, C16, C17, C18: 100n, symbol Device:C
- removed D1: LED, symbol Device:LED
- removed IC1: BMP390, BMP390, symbol BMP390:BMP390
- removed R2: 1k, symbol Device:R
- removed R3, R4, R5: 56k, symbol Device:R
- removed U2: AMS1117-3.3, Package_TO_SOT_SMD:SOT-223-3_TabPin2, symbol Regulator_Linear:AMS1117-3.3
- removed U3: BMI088, BMI088:PQFN50P450X300X100-16N, symbol BMI088:BMI088
- removed U4: LSM6DSLTR, LSM6DSLTR:PQFN50P300X250X86-14N, symbol LSM6DSLTR:LSM6DSLTR
- removed U5: BMM150, Package_CSP:WLCSP-12_1.56x1.56mm_P0.4mm, symbol Sensor_Magnetic:BMM150
Connections:
- net BAR_CLK: now also U1.34 (PB13)
- net BAR_INT: now also U1.33 (PB12)
- net BAR_MISO: now also U1.35 (PB14)
- net BAR_MOSI: now also U1.36 (PB15)
- net IMU1_CSB_ACCEL: no longer U1.11 (PC3)
- net IMU1_INT_ACCEL: now also U1.11 (PC3)
- net BAR_CSB: now reaches U1.30 (PB11)
- net VBUS renamed +5V
- no-connect marks 4 -> 2
Other:
- added sheet Power (Power.kicad_sch)
- added sheet Sensors (Sensors.kicad_sch)
- note removed: "Pressure Sensor"
- note removed: "Primary IMU"
- moved on the sheet: C1, C10, C11, C12, C2, C3, C4, C5, C6, C7, C8, C9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

Commit message: update
Parts:
- removed C1, C10, C2, C3, C4, C5: 100n, symbol Device:C
- removed C11, C12: 10p, symbol Device:C
- removed C6: 10u, symbol Device:C
- removed C7: 10n, symbol Device:C
- removed C8, C9: 1u, symbol Device:C
- removed FB1: 120R, symbol Device:FerriteBead
- removed J1: USB_B_Micro, symbol Connector:USB_B_Micro
- removed J2: Conn_01x04_Pin, symbol Connector:Conn_01x04_Pin
- removed R1: 10k, symbol Device:R
- removed SW1: SW_SPDT, symbol Switch:SW_SPDT
- removed U1: STM32F405RGTx, Package_QFP:LQFP-64_10x10mm_P0.5mm, symbol MCU_ST_STM32F4:STM32F405RGTx
- removed Y1: 16MHz, symbol Device:Crystal_GND24
- added C27, C33, C34, C35, C36, C37, C41, C43: 100n, symbol Device:C
- added C28, C29: 2u2, symbol Device:C
- added C30, C31: 10p, symbol Device:C
- added C32: 10u, symbol Device:C
- added C38: 10n, symbol Device:C
- added C39, C40, C42: 1u, symbol Device:C
- added D3: SS14, Diode_SMD:D_SMA, symbol Diode:SS14
- added FB2: 120R, symbol Device:FerriteBead
- added FB4: FerriteBead, symbol Device:FerriteBead
- added J4: Conn_01x05, symbol Connector_Generic:Conn_01x05
- added J7: USB_B_Micro, symbol Connector:USB_B_Micro
- added MPU: STM32H753VITx, Package_QFP:LQFP-100_14x14mm_P0.5mm, symbol MCU_ST_STM32H7:STM32H753VITx
- added R12: 10k, symbol Device:R
- added R13: 47, symbol Device:R
- added R14, R15, R16, R17: 4k7, symbol Device:R
- added SW2: SW_SPDT, symbol Switch:SW_SPDT
- added Y2: 16MHz, symbol Device:Crystal_GND24
Connections:
- net +3.3V: now also C32.1, C33.1, C34.1, C35.1, C36.1, C37.1, C40.1, C41.1, FB2.2, MPU.100 (VDD), MPU.11 (VDD), MPU.27 (VDD), MPU.50 (VDD), MPU.6 (VBAT), MPU.75 (VDD), R14.1, R15.1, R16.1, R17.1, SW2.3 (C)
- net +3.3VA: now also C38.1, C39.1, FB2.1, J4.1 (Pin_1), MPU.21 (VDDA), R13.1
- net +5V: now also FB4.2
- net GND: now also C27.2, C28.2, C29.2, C30.2, C31.2, C32.2, C33.2, C34.2, C35.2, C36.2, C37.2, C38.2, C39.2, C40.2, C41.2, C42.2, C43.2, J4.5 (Pin_5), J7.5 (GND), MPU.10 (VSS), MPU.19 (VSSA), MPU.26 (VSS), MPU.49 (VSS), MPU.74 (VSS), MPU.99 (VSS), SW2.1 (A), Y2.2, Y2.4
- new net: D3.2 (A), J7.1 (VBUS)
- new net: C28.1, MPU.48 (VCAP)
- new net: D3.1 (K), FB4.1
- new net: C29.1, MPU.73 (VCAP)
- new net BOOT0_MPU: MPU.94 (BOOT0), R12.2
- new net HSE_IN_MPU: C30.1, MPU.12 (PH0), Y2.1
- new net HSE_OUT_MPU: C31.1, MPU.13 (PH1), Y2.3
- new net I2C1_SCL_MPU: MPU.92 (PB6), R15.2
- new net I2C1_SDA_MPU: MPU.93 (PB7), R14.2
- new net I2C2_SCL_MPU: MPU.46 (PB10), R17.2
- new net I2C2_SDA_MPU: MPU.47 (PB11), R16.2
- new net NRST_MPU: C27.1, J4.4 (Pin_4), MPU.14 (NRST)
- new net Pyro_1: MPU.59 (PD12)
- new net Pyro_2: MPU.60 (PD13)
- new net Pyro_3: MPU.61 (PD14)
- new net Pyro_4: MPU.62 (PD15)
- new net SPI1_CS_MPU: MPU.28 (PA4)
- new net SPI1_MISO_MPU: MPU.30 (PA6)
- new net SPI1_MOSI_MPU: MPU.31 (PA7)
- new net SPI1_SCK_MPU: MPU.29 (PA5)
- new net SWCLK_MPU: J4.3 (Pin_3), MPU.77 (PA15)
- new net SWDIO_MPU: J4.2 (Pin_2), MPU.76 (PA14)
- new net SW_BOOT0_NAV: R12.1, SW2.2 (B)
- new net USART1_RX_MPU: MPU.54 (PB15)
- new net USART1_TX_MPU: MPU.53 (PB14)
- new net USB_D+_MPU: J7.3 (D+), MPU.71 (PA12)
- new net USB_D-_MPU: J7.2 (D-), MPU.70 (PA11)
- new net VREF+_MPU: C42.1, C43.1, MPU.20 (VREF+), R13.2
Other:
- sheet Power renamed Power Management
- sheet Sensors renamed Sensors and NavPeripherals
- added sheet MPU Peripherals (MPU_Peripherals.kicad_sch)
- added sheet Navigation Processing Unit (NAVComputer_sch.kicad_sch)
- note added: "DEBUG_NAV"
- note added: "HIGH SPEED EXTERNAL CRYSTAL"
- note added: "I2C Pullups"
- note added: "Main Processing Unit"
- note added: "USB_MPU"
- note added: "VDDA FILTER"
- note added: "VREF+ FILTER"
- note removed: "USB DIFFERENTIAL PAIR"
- title: (none) -> Main Processing Unit

Commit message: Refactor code structure for improved readability and maintainability
Parts:
- added D4, D5: LED_RED, symbol Device:LED
- added D6, D7: LED_GREEN, symbol Device:LED
- added R34, R35, R36, R37: 220, symbol Device:R
Connections:
- net +3.3VA: no longer R13.1
- net GND: now also R34.2, R35.2, R36.2, R37.2
- net SWCLK_MPU: now also MPU.76 (PA14); no longer MPU.77 (PA15)
- net SWDIO_MPU: now also MPU.72 (PA13); no longer MPU.76 (PA14)
- net USART1_RX_MPU: now also MPU.69 (PA10); no longer MPU.54 (PB15)
- net USART1_TX_MPU: now also MPU.68 (PA9); no longer MPU.53 (PB14)
- net SD_CLK: now reaches MPU.16 (PC1)
- net SD_CMD: now reaches MPU.22 (PA0)
- net SD_DAT2: now reaches MPU.89 (PB3)
- net SD_DAT3: now reaches MPU.90 (PB4)
- new net: D4.1 (K), R34.1
- new net: D7.1 (K), R37.1
- new net: D6.1 (K), R36.1
- new net: D5.1 (K), R35.1
- new net LED1_MPU: D4.2 (A)
- new net LED2_MPU: D5.2 (A)
- new net LED3_MPU: D6.2 (A)
- new net LED4_MPU: D7.2 (A)
- new net SD_DAT0: MPU.53 (PB14)
- new net SD_DAT1: MPU.54 (PB15)
- new net SD_DET: MPU.77 (PA15)
- new net VDDA_MPU: R13.1
Other:
- note added: "Status LEDs"
- moved on the sheet: C30, C31, D3, FB4, J4, J7, R14, R15, R16, R17, Y2

Commit message: Add lock file for ALBERT_FLIGHTCOMPUTER PCB design
Parts:
- removed C32: 10u, symbol Device:C
- removed C39, C40, C42: 1u, symbol Device:C
- removed J7: USB_B_Micro, symbol Connector:USB_B_Micro
- added C5, C6, C8: 1u, Capacitor_Tantalum_SMD:CP_EIA-1608-10_AVX-L, symbol Device:C_Polarized
- added C7: 10u, Capacitor_Tantalum_SMD:CP_EIA-1608-10_AVX-L, symbol Device:C_Polarized
- added J2: USB_C_Receptacle_USB2.0_14P, Connector_USB:USB_C_Receptacle_HRO_TYPE-C-31-M-12, symbol Connector:USB_C_Receptacle_USB2.0_14P
- added R39, R40: 5k1, Resistor_SMD:R_0402_1005Metric, symbol Device:R
- C1: renamed from C27; footprint (none) -> Capacitor_SMD:C_0402_1005Metric
- C10: renamed from C33; footprint (none) -> Capacitor_SMD:C_0402_1005Metric
- C11: renamed from C34; footprint (none) -> Capacitor_SMD:C_0402_1005Metric
- C12: renamed from C35; footprint (none) -> Capacitor_SMD:C_0402_1005Metric
- C13: renamed from C30; footprint (none) -> Capacitor_SMD:C_0402_1005Metric
- C14: renamed from C36; footprint (none) -> Capacitor_SMD:C_0402_1005Metric
- C15: renamed from C37; footprint (none) -> Capacitor_SMD:C_0402_1005Metric
- C16: renamed from C31; footprint (none) -> Capacitor_SMD:C_0402_1005Metric
- C17: renamed from C41; footprint (none) -> Capacitor_SMD:C_0402_1005Metric
- C2: renamed from C28; footprint (none) -> Capacitor_SMD:C_0805_2012Metric
- C3: renamed from C29; footprint (none) -> Capacitor_SMD:C_0805_2012Metric
- C4: renamed from C38; footprint (none) -> Capacitor_SMD:C_0402_1005Metric
- C9: renamed from C43; footprint (none) -> Capacitor_SMD:C_0402_1005Metric
- D1: renamed from D4; footprint (none) -> LED_SMD:LED_0603_1608Metric
- D2: renamed from D5; footprint (none) -> LED_SMD:LED_0603_1608Metric
- D3: renamed from D6; footprint (none) -> LED_SMD:LED_0603_1608Metric
- D4: renamed from D7; footprint (none) -> LED_SMD:LED_0603_1608Metric
- FB1: renamed from FB2; footprint (none) -> Inductor_SMD:L_0603_1608Metric
- FB2: renamed from FB4; footprint (none) -> Inductor_SMD:L_0603_1608Metric
- J1: renamed from J4; footprint (none) -> Connector_PinHeader_2.54mm:PinHeader_1x05_P2.54mm_Vertical
- R1: renamed from R34; footprint (none) -> Resistor_SMD:R_0402_1005Metric
- R10: renamed from R12; footprint (none) -> Resistor_SMD:R_0402_1005Metric
- R2: renamed from R14; footprint (none) -> Resistor_SMD:R_0402_1005Metric
- R3: renamed from R15; footprint (none) -> Resistor_SMD:R_0402_1005Metric
- R4: renamed from R35; footprint (none) -> Resistor_SMD:R_0402_1005Metric
- R5: renamed from R16; footprint (none) -> Resistor_SMD:R_0402_1005Metric
- R6: renamed from R36; footprint (none) -> Resistor_SMD:R_0402_1005Metric
- R7: renamed from R17; footprint (none) -> Resistor_SMD:R_0402_1005Metric
- R8: renamed from R37; footprint (none) -> Resistor_SMD:R_0402_1005Metric
- R9: renamed from R13; footprint (none) -> Resistor_SMD:R_0402_1005Metric
- SW1: renamed from SW2; footprint (none) -> Button_Switch_SMD:SW_SPDT_PCM12
- Y1: renamed from Y2; footprint (none) -> Crystal:Crystal_SMD_3225-4Pin_3.2x2.5mm
- renumbered D3 to D5, MPU to MPU1
Connections:
- net +3.3V: now also J1.1 (Pin_1), C6.1, C7.1
- net GND: now also C5.2, C6.2, C7.2, C8.2, J2.A1 (GND), J2.A12 (GND), J2.B1 (GND), J2.B12 (GND), J2.S1 (SHIELD), R39.2, R40.2
- net LED1_MPU: now also MPU1.81 (PD0)
- net LED2_MPU: now also MPU1.82 (PD1)
- net LED3_MPU: now also MPU1.83 (PD2)
- net LED4_MPU: now also MPU1.84 (PD3)
- net VDDA_MPU: now also C4.1, FB1.1, MPU1.21 (VDDA), C5.1
- net VREF+_MPU: now also C8.1
- net at D5.2 (A): now also J2.A4 (VBUS), J2.A9 (VBUS), J2.B4 (VBUS), J2.B9 (VBUS)
- net SPI4_SCK_MPU: now reaches MPU1.1 (PE2)
- net SPI2_MISO_MPU: now reaches MPU1.17 (PC2_C)
- net SPI2_MOSI_MPU: now reaches MPU1.18 (PC3_C)
- net USART2_TX_MPU: now reaches MPU1.24 (PA2)
- net USART2_RX_MPU: now reaches MPU1.25 (PA3)
- net SPI4_NSS_MPU: now reaches MPU1.3 (PE4)
- net SPI2_DIO0_MPU: now reaches MPU1.32 (PC4)
- net SPI2_DIO2_MPU: now reaches MPU1.33 (PC5)
- net LORA_RST_MPU: now reaches MPU1.34 (PB0)
- net GPIO1_MPU: now reaches MPU1.37 (PE7)
- net GPIO2_MPU: now reaches MPU1.38 (PE8)
- net GPIO3_MPU: now reaches MPU1.39 (PE9)
- net SPI4_MISO_MPU: now reaches MPU1.4 (PE5)
- net GPIO4_MPU: now reaches MPU1.40 (PE10)
- net GPIO5_MPU: now reaches MPU1.41 (PE11)
- net GPIO6_MPU: now reaches MPU1.42 (PE12)
- net GPIO7_MPU: now reaches MPU1.43 (PE13)
- net GPIO8_MPU: now reaches MPU1.44 (PE14)
- net GPIO9_MPU: now reaches MPU1.45 (PE15)
- net SPI4_MOSI_MPU: now reaches MPU1.5 (PE6)
- net SPI2_NSS_MPU: now reaches MPU1.51 (PB12)
- net SPI2_SCK_MPU: now reaches MPU1.52 (PB13)
- net USART3_TX_MPU: now reaches MPU1.55 (PD8)
- net USART3_RX_MPU: now reaches MPU1.56 (PD9)
- net INT1_MPU: now reaches MPU1.57 (PD10)
- net INT2_MPU: now reaches MPU1.58 (PD11)
- net GPIO10_MPU: now reaches MPU1.63 (PC6)
- net GPIO11_MPU: now reaches MPU1.64 (PC7)
- net GPIO12_MPU: now reaches MPU1.65 (PC8)
- removed net +3.3VA: C4.1, FB1.1, J1.1 (Pin_1), MPU1.21 (VDDA)
- net Pyro_1 renamed Pyro_4_MPU
- net Pyro_2 renamed Pyro_3_MPU
- net Pyro_3 renamed Pyro_2_MPU
- net Pyro_4 renamed Pyro_1_MPU
- net SD_CLK renamed SD_CLK_MPU
- net SD_CMD renamed SD_CMD_MPU
- net SD_DAT0 renamed SD_DAT0_MPU
- net SD_DAT1 renamed SD_DAT1_MPU
- net SD_DAT2 renamed SD_DAT2_MPU
- net SD_DAT3 renamed SD_DAT3_MPU
- net SD_DET renamed SD_DET_MPU
- net USB_D+_MPU renamed USB_MPU_D+
- net USB_MPU_D+: now also J2.A6 (D+), J2.B6 (D+)
- net USB_D-_MPU renamed USB_MPU_D-
- net USB_MPU_D-: now also J2.A7 (D-), J2.B7 (D-)
- new net: J2.B5 (CC2), R39.1
- new net: J2.A5 (CC1), R40.1
- no-connect marks 2 -> 22
Other:
- sheet Navigation Processing Unit renamed NAV
- added sheet GPS & LORA (GPS & LORA.kicad_sch)
- company: (none) -> ALBERT AEROSPACE
- moved on the sheet: C1, C13, C16, C2, C3, C9, D1, D2, D3, D4, D5, FB2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

Commit message: Add production files and update project lock file
- Added new production IT1 zip file for ALBERT_FLIGHTCOMPUTER.
- Removed obsolete test zip file from production directory.
- Created a lock file for the KiCad schematic with user and hostname information.
Parts:
- removed C5, C6, C8: 1u, Capacitor_Tantalum_SMD:CP_EIA-1608-10_AVX-L, symbol Device:C_Polarized
- removed C7: 10u, Capacitor_Tantalum_SMD:CP_EIA-1608-10_AVX-L, symbol Device:C_Polarized
- added C5, C6, C8: 1u, Capacitor_SMD:C_0805_2012Metric, symbol Device:C
- added C7: 10u, Capacitor_SMD:C_0805_2012Metric, symbol Device:C
- added U9: USBLC6-2SC6, Package_TO_SOT_SMD:SOT-23-6, symbol Power_Protection:USBLC6-2SC6
- C1, C10, C11, C12, C14, C15, C17, C9: LCSC (none) -> C1525
- C13, C16: LCSC (none) -> C32949
- C2, C3: LCSC (none) -> C377773
- C4: LCSC (none) -> C15195
- D5: LCSC (none) -> C2480
- FB1: value 120R -> 100R; LCSC (none) -> C15957
- FB2: value FerriteBead -> 100R; footprint Inductor_SMD:L_0603_1608Metric -> Inductor_SMD:L_0805_2012Metric; LCSC (none) -> C15957
- J2: LCSC (none) -> C165948
- MPU1: value STM32H753VITx -> STM32H753VIT6; LCSC (none) -> C730206; Manufacturer (none) -> STMicroelectronics; Manufacturer Part Number (none) -> STM32H753VIT6
- R1, R4, R6, R8: LCSC (none) -> C25091
- R10: LCSC (none) -> C25744
- R2, R3, R5, R7: LCSC (none) -> C25900
- R39, R40: LCSC (none) -> C25905
- R9: value 47 -> 22; LCSC (none) -> C25092
- SW1: LCSC (none) -> C221841
- Y1: LCSC (none) -> C13738
Connections:
- net +3.3V: now also C6.1, C7.1
- net GND: now also C5.2, C6.2, C7.2, C8.2, U9.2 (GND)
- net USB_MPU_D+: now also U9.4 (I/O2); no longer J2.A6 (D+), J2.B6 (D+)
- net USB_MPU_D-: now also U9.6 (I/O1); no longer J2.A7 (D-), J2.B7 (D-)
- net VDDA_MPU: now also C5.1
- net VREF+_MPU: now also C8.1
- net at D5.2 (A), J2.A4 (VBUS), J2.A9 (VBUS)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: now also U9.5 (VBUS)
- new net ESD_MPU_D+: J2.A6 (D+), J2.B6 (D+), U9.3 (I/O2)
- new net ESD_MPU_D-: J2.A7 (D-), J2.B7 (D-), U9.1 (I/O1)
Other:
- moved on the sheet: D5, FB2, R39, R40
