File: 3_Flight_Computer/PCB/ALBERT_FLIGHTCOMPUTER/ALBERT_FLIGHTCOMPUTER.kicad_sch (KiCad schematic)
At the start: 42 parts, among them J1 Conn_01x05, J2 USB_C_Receptacle_USB2.0_14P, SW1 SW_SPDT, U9 USBLC6-2SC6, Y1 16MHz

Commit message: Die EU ruft die Renaissance der Atomkraft aus – und Österreich schreit: "Schleich di!"
Other:
- company: ALBERT AEROSPACE -> ALBERT AERO
Changed lines of the file:
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@@
 		(date "2025-11-10")
 		(rev "0.1")
-		(company "ALBERT AEROSPACE")
+		(company "ALBERT AERO")
 	)
 	(rectangle
