File: 3_Flight_Computer/PCB/ALBERT_FLIGHTCOMPUTER/GPS & LORA.kicad_sch (KiCad schematic)
At the start: 15 parts, among them J18 5-1814400-2, J19 5-1814400-2, U7 RFM95W-868S2, U8 ZOE-M8Q, Y3 CM7V-T1A-32.768KHZ-6PF-20PPM-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

Commit message: update pcb
Other:
- title: RF -> GPS & LORA
Changed lines of the file:
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@@
 	(paper "A4")
 	(title_block
-		(title "RF")
+		(title "GPS & LORA")
 		(date "2025-11-10")
 		(rev "0.1")

Commit message: Add production files and update project lock file
- Added new production IT1 zip file for ALBERT_FLIGHTCOMPUTER.
- Removed obsolete test zip file from production directory.
- Created a lock file for the KiCad schematic with user and hostname information.
Parts:
- removed Y3: CM7V-T1A-32.768KHZ-6PF-20PPM-TA-QC, CMV-T1A-32.768KHZ:CM7V32768TBQA020, symbol CM7V-T1A-32_768KHZ-6PF-20PPM-T:CM7V-T1A-32.768KHZ-6PF-20PPM-TA-QC
- added Y3: 32.768kHz, Crystal:Crystal_SMD_MicroCrystal_CC7V-T1A-2Pin_3.2x1.5mm, symbol Device:Crystal
- C60, C62: LCSC (none) -> C1525
- C61: LCSC (none) -> C1746
- C63: LCSC (none) -> C478452
- D8: LCSC (none) -> C233388
- FB5: LCSC (none) -> C21516
- J18, J19: LCSC (none) -> C3174972
- JP1, U7: now left out of the parts list
- L3: LCSC (none) -> C113100
- R46: LCSC (none) -> C25744
- R47: LCSC (none) -> C25077
- U8: LCSC (none) -> C7398634
Connections:
- net at U8.J7 (RTC_I): now also Y3.2
- net at U8.J8 (RTC_O): now also Y3.1
