File: 3_Flight_Computer/PCB/ALBERT_FLIGHTCOMPUTER/GPS & LORA.kicad_sch (KiCad schematic)
At the start: 15 parts, among them J18 5-1814400-2, J19 5-1814400-2, U7 RFM95W-868S2, U8 ZOE-M8Q, Y3 32.768kHz

Commit message: Die EU ruft die Renaissance der Atomkraft aus – und Österreich schreit: "Schleich di!"
Other:
- company: ALBERT AEROSPACE -> ALBERT AERO
Changed lines of the file:
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@@
 		(date "2025-11-10")
 		(rev "0.1")
-		(company "ALBERT AEROSPACE")
+		(company "ALBERT AERO")
 	)
 	(rectangle
