File: 3_Flight_Computer/PCB/ALBERT_FLIGHTCOMPUTER/MPU_Peripherals.kicad_sch (KiCad schematic)
At the start: 38 parts, among them IC1 PCA9685PW,118, IC2 W25N01GVZEIG, J10 Conn_01x06, J12 Conn_02x08_Odd_Even, J13 HXPZ2.54-3x8PZZ1, J3 Screw_Terminal_01x02, J4 Screw_Terminal_01x02, J5 Screw_Terminal_01x02, J6 Screw_Terminal_01x02, J7 Micro_SD_Card_Det2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

Commit message: Pregnant Women, DON’T USE TYLENOL UNLESS ABSOLUTELY NECESSARY, DON’T GIVE TYLENOL TO YOUR YOUNG CHILD FOR VIRTUALLY ANY REASON, BREAK UP THE MMR SHOT INTO THREE TOTALLY SEPARATE SHOTS (NOT MIXED!), TAKE CHICKEN P SHOT SEPARATELY, TAKE HEPATITAS B SHOT AT 12 YEARS OLD, OR OLDER, AND, IMPORTANTLY, TAKE VACCINE IN 5 SEPARATE MEDICAL VISITS! President DJT
Parts:
- removed J13: HXPZ2.54-3x8PZZ1, HXPZ2.54-3x8PZZ:HX PZ2.54-3x8P ZZ, symbol HXPZ2.54-3x8PZZ:HXPZ2.54-3x8PZZ
- added J13: Conn_02x08_Odd_Even, Connector_PinHeader_2.54mm:PinHeader_2x08_P2.54mm_Vertical, symbol Connector_Generic:Conn_02x08_Odd_Even
- added J20: Conn_01x08, Connector_PinHeader_2.54mm:PinHeader_1x08_P2.54mm_Vertical, symbol Connector_Generic:Conn_01x08
Connections:
- net GND: now also J13.1 (Pin_1), J13.11 (Pin_11), J13.13 (Pin_13), J13.15 (Pin_15), J13.3 (Pin_3), J13.5 (Pin_5), J13.7 (Pin_7), J13.9 (Pin_9)
- net PWM_00: now also J20.1 (Pin_1)
- net PWM_01: now also J20.2 (Pin_2)
- net PWM_02: now also J20.3 (Pin_3)
- net PWM_03: now also J20.4 (Pin_4)
- net PWM_04: now also J20.5 (Pin_5)
- net PWM_05: now also J20.6 (Pin_6)
- net PWM_06: now also J20.7 (Pin_7)
- net PWM_07: now also J20.8 (Pin_8)
- net VBAT: now also J13.10 (Pin_10), J13.12 (Pin_12), J13.14 (Pin_14), J13.16 (Pin_16), J13.2 (Pin_2), J13.4 (Pin_4), J13.6 (Pin_6), J13.8 (Pin_8)
Changed lines of the file:
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@@
-	)
-	(symbol
-		(lib_id "HXPZ2.54-3x8PZZ:HXPZ2.54-3x8PZZ")
-		(at 212.09 44.45 0)
-		(unit 1)
-		(exclude_from_sim no)
-		(in_bom yes)
-		(on_board yes)
-		(dnp no)
-		(property "Reference" "J13"
-			(at 227.076 16.764 0)
-			(effects
-				(font
-					(size 1.27 1.27)
-				)
-			)
-		)
-		(property "Value" "HXPZ2.54-3x8PZZ1"
-			(at 235.204 19.304 0)
-			(effects
-				(font
-					(size 1.27 1.27)
-				)
-			)
-		)
-		(property "Footprint" "HXPZ2.54-3x8PZZ:HX PZ2.54-3x8P ZZ"
-			(at 212.09 44.45 0)
-			(effects
-				(font
-					(size 1.27 1.27)
-				)
-				(hide yes)
-			)
-		)
-		(property "Datasheet" ""
-			(at 212.09 44.45 0)
-			(effects
-				(font
-					(size 1.27 1.27)
-				)
-				(hide yes)
-			)
-		)
-		(property "Description" ""
-			(at 212.09 44.45 0)
-			(effects
-				(font
-					(size 1.27 1.27)
-				)
-				(hide yes)
-			)
-		)
-		(property "LCSC" "C32713295"
-			(at 212.09 44.45 0)
-			(effects
-				(font
-					(size 1.27 1.27)
-				)
-				(hide yes)
-			)
-		)
-		(pin "24"
-		)
-		(pin "2"
-		)
-		(pin "22"
-		)
-		(pin "5"
-		)
-		(pin "19"
-		)
-		(pin "23"
-		)
-		(pin "20"
-		)
-		(pin "17"
-		)
-		(pin "14"
-		)
-		(pin "10"
-		)
-		(pin "7"
-		)
-		(pin "16"
-		)
-		(pin "13"
-		)
-		(pin "21"
-		)
-		(pin "18"
-		)
-		(pin "12"
-		)
-		(pin "15"
-		)
-		(pin "9"
-		)
-		(pin "3"
-		)
-		(pin "6"
-		)
-		(pin "1"
-		)
-		(pin "11"
-		)
-		(pin "8"
-		)
-		(pin "4"
-		)
-		(instances
-			(project ""
-				(path "/caf1b85f-a91d-4c85-9df1-65f9ebc85027/1edee9cd-27d7-479a-992c-cbc714ec1449"
-					(reference "J13")
-					(unit 1)
-				)
-			)
-		)
 	)
 	(symbol
@@
 	)
 	(symbol
+		(lib_id "Connector_Generic:Conn_02x08_Odd_Even")
+		(at 210.82 31.75 0)
+		(unit 1)
+		(exclude_from_sim no)
+		(in_bom yes)
+		(on_board yes)
+		(dnp no)
+		(fields_autoplaced yes)
+		(property "Reference" "J13"
+			(at 212.09 17.78 0)
+			(effects
+				(font
+					(size 1.27 1.27)
+				)
+			)
+		)
+		(property "Value" "Conn_02x08_Odd_Even"
+			(at 212.09 20.32 0)
+			(effects
+				(font
+					(size 1.27 1.27)
+				)
+			)
+		)
+		(property "Footprint" "Connector_PinHeader_2.54mm:PinHeader_2x08_P2.54mm_Vertical"
+			(at 210.82 31.75 0)
+			(effects
+				(font
+					(size 1.27 1.27)
+				)
+				(hide yes)
+			)
+		)
+		(property "Datasheet" "~"
+			(at 210.82 31.75 0)
+			(effects
+				(font
+					(size 1.27 1.27)
+				)
+				(hide yes)
+			)
+		)
+		(property "Description" "Generic connector, double row, 02x08, odd/even pin numbering scheme (row 1 odd numbers, row 2 even numbers), script generated (kicad-library-utils/schlib/autogen/connector/)"
+			(at 210.82 31.75 0)
+			(effects
+				(font
+					(size 1.27 1.27)
+				)
+				(hide yes)
+			)
+		)
+		(pin "10"
+		)
+		(pin "12"
+		)
+		(pin "14"
+		)
+		(pin "16"
+		)
+		(pin "3"
+		)
+		(pin "13"
+		)
+		(pin "1"
+		)
+		(pin "4"
+		)
+		(pin "6"
+		)
+		(pin "8"
+		)
+		(pin "5"
+		)
+		(pin "11"
+		)
+		(pin "2"
+		)
+		(pin "9"
+		)
+		(pin "15"
+		)
+		(pin "7"
+		)
+		(instances
+			(project "ALBERT_FLIGHTCOMPUTER"
+				(path "/caf1b85f-a91d-4c85-9df1-65f9ebc85027/1edee9cd-27d7-479a-992c-cbc714ec1449"
+					(reference "J13")
+					(unit 1)
+				)
+			)
+		)
+	)
+	(symbol
 		(lib_id "power:+3.3V")
 		(at 180.34 107.95 0)
@@
 					(unit 1)
 				)
+			)
+		)
+	)
+	(symbol
+		(lib_id "Connector_Generic:Conn_01x08")
+		(at 240.03 31.75 0)
+		(unit 1)
+		(exclude_from_sim no)
+		(in_bom yes)
+		(on_board yes)
+		(dnp no)
+		(property "Reference" "J20"
+			(at 235.204 18.034 0)
+			(effects
+				(font
+					(size 1.27 1.27)
+				)
+				(justify left)
+			)
+		)
+		(property "Value" "Conn_01x08"
+			(at 230.632 20.066 0)
+			(effects
+				(font
+					(size 1.27 1.27)
+				)
+				(justify left)
+			)
+		)
+		(property "Footprint" "Connector_PinHeader_2.54mm:PinHeader_1x08_P2.54mm_Vertical"
+			(at 240.03 31.75 0)
+			(effects
+				(font
+					(size 1.27 1.27)
+				)
+				(hide yes)
+			)
+		)
+		(property "Datasheet" "~"
+			(at 240.03 31.75 0)
+			(effects
+				(font
+					(size 1.27 1.27)
+				)
+				(hide yes)
+			)
+		)
+		(property "Description" "Generic connector, single row, 01x08, script generated (kicad-library-utils/schlib/autogen/connector/)"
+			(at 240.03 31.75 0)
+			(effects
+				(font
+					(size 1.27 1.27)
+				)
+				(hide yes)
+			)
+		)
+		(pin "1"
+		)
+		(pin "2"
+		)
+		(pin "3"
+		)
+		(pin "4"
+		)
+		(pin "5"
+		)
+		(pin "6"
+		)
+		(pin "7"
+		)
+		(pin "8"
+		)
+		(instances
+			(project "ALBERT_FLIGHTCOMPUTER"
+				(path "/caf1b85f-a91d-4c85-9df1-65f9ebc85027/1edee9cd-27d7-479a-992c-cbc714ec1449"
+					(reference "J20")
+					(unit 1)
+				)

Commit message: Die EU ruft die Renaissance der Atomkraft aus – und Österreich schreit: "Schleich di!"
Other:
- company: ALBERT AEROSPACE -> ALBERT AERO
Changed lines of the file:
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@@
 		(date "2025-11-10")
 		(rev "0.1")
-		(company "ALBERT AEROSPACE")
+		(company "ALBERT AERO")
 	)
 	(rectangle
