File: 3_Flight_Computer/PCB/ALBERT_FLIGHTCOMPUTER/Power.kicad_sch (KiCad schematic)
At the start: 8 parts, among them J3 XT60-M, U2 AMS1117-3.3, U6 TPS54308

Commit message: Refactor code structure for improved readability and maintainability
Parts:
- added C19: 10u, symbol Device:C
- added C20, C21, C24: 100n, symbol Device:C
- added C22, C23: 22u, symbol Device:C
- added L1: 10u, symbol Device:L_Iron_Small
- added R10: 100k, symbol Device:R
- added R11: 13k7, symbol Device:R
- added R7: 511k, symbol Device:R
- added R8: 105k, symbol Device:R
- added R9: 49.9, symbol Device:R
- added U7: INA219AxDCN, Package_TO_SOT_SMD:SOT-23-8, symbol Sensor_Energy:INA219AxDCN
Connections:
- net +3.3V: now also C24.1, U7.4 (VS)
- net +5V: now also C22.1, C23.1, L1.2, R9.1
- net GND: now also U6.1 (GND), C19.2, C20.2, C22.2, C23.2, C24.2, R11.2, R8.2, U7.3 (GND), U7.7 (A0), U7.8 (A1)
- net at U6.2 (SW): now also C21.2, L1.1
- net at U6.3 (VIN): now also C19.1, C20.1, R7.1
- net at U6.4 (FB): now also R10.2, R11.1
- net at U6.5 (EN): now also R7.2, R8.1
- net at U6.6 (BOOT): now also C21.1
- net VIN+ renamed IN+
- net IN+: now also U7.1 (IN+)
- net VIN- renamed IN-
- net IN-: now also U7.2 (IN-)
- new net: R10.1, R9.2
Other:
- note added: "5V/3,3V Converter"
- note added: "Buck Converter 12V/5V"
- note added: "C19 - ceramic C21 - ceramic pay attention to the max voltage ratings of the caps"
- note added: "Voltage & Current Sensing"
- moved on the sheet: C13, C14, D1, R2, U2, U6

Commit message: update
Parts:
- added C44: 2n2, symbol Device:C
- added IC2: TPS621351RGXR, TPS621361RGXT, symbol TPS621351RGXR:TPS621351RGXR
- added L2: 1u, symbol Device:L_Iron_Small
- C19: value 10u -> 6u8
- C20: value 100n -> 10u
- C22: value 22u -> 10u
- C23: value 22u -> 47u
- L1: value 10u -> 15u
- R7: value 511k -> 1M1
- R8: value 105k -> 100k
- R9: value 49.9 -> 100k
Connections:
- net +5V: now also R10.1; no longer C22.1, R9.1
- net GND: now also C44.2, IC2.10 (MODE), IC2.11 (VSEL), IC2.3 (GND), IC2.4 (FB2)
- net +8V4: now reaches C20.1, R7.1
- net +8V4: now also R9.2, IC2.6 (VOS), L2.2; no longer C19.1, U6.3 (VIN)
- net at R7.2, R8.1: now also IC2.5 (FB); no longer U6.5 (EN)
- net I2C2_SCL_MPU: now reaches U7.5 (SCL)
- net I2C2_SDA_MPU: now reaches U7.6 (SDA)
- net IN- renamed VBAT
- net VBAT: now also C19.1, C22.1, U6.3 (VIN), IC2.1 (VIN), IC2.8 (EN)
- new net: C44.1, IC2.9 (SS/TR)
- new net: IC2.2 (SW), L2.1
- new net: IC2.7 (PG), R9.1
- no-connect marks 0 -> 1
Other:
- note added: "Buck Converter DOS 12V/8,4V"
- note added: "Buck Converter UNO 12V/5V"
- note added: "I2C ADDRESS: 0x40"
- note added: "Shunt: R6 == 10mOhm 1W 2512"
- note removed: "Buck Converter 12V/5V"
- title: (none) -> Power Management
- moved on the sheet: C13, C14, C19, C21, C23, C24, D1, J3, L1, R10, R11, R2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

Commit message: Refactor code structure for improved readability and maintainability
Parts:
- C19: value 6u8 -> 10u
- D1: value LED -> LED_GREEN
- L1: value 15u -> 10u
- R11: value 13k7 -> 22k
- R2: value 1k -> 220
Connections:
- net +3.3V: now also C23.1, L1.2, R10.1
- net +5V: no longer C23.1, L1.2, R10.1
Other:
- note added: "Buck Converter UNO 12V/3V3"
- note added: "Tantalum"
- note removed: "Buck Converter UNO 12V/5V"
Changed lines of the file:
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@@
 		)
 	)
+	(text "Tantalum\n"
+		(exclude_from_sim no)
+		(at 101.6 97.536 0)
+		(effects
+			(font
+				(size 1.27 1.27)
+			)
+		)
+	)
 	(text "C19 - ceramic\nC21 - ceramic\n\npay attention to the max voltage ratings of the caps\n"
 		(exclude_from_sim no)
@@
 		)
 	)
-	(text "Buck Converter UNO 12V/5V\n"
+	(text "Buck Converter UNO 12V/3V3\n"
 		(exclude_from_sim no)
 		(at 143.764 78.74 0)
@@
 	(wire
 		(pts
+			(xy 240.03 36.83) (xy 240.03 38.1)
+		)
+		(stroke
+			(width 0)
+			(type default)
+		)
+	)
+	(wire
+		(pts
 			(xy 48.26 86.36) (xy 48.26 90.17)
 		)
@@
 	)
 	(global_label "I2C2_SDA_MPU"
-		(shape input)
+		(shape bidirectional)
 		(at 86.36 129.54 0)
 		(fields_autoplaced yes)
@@
 		)
 		(property "Intersheetrefs" "${INTERSHEET_REFS}"
-			(at 103.1942 129.54 0)
+			(at 104.3055 129.54 0)
 			(effects
 				(font
@@
 	)
 	(symbol
-		(lib_id "power:+5V")
-		(at 240.03 38.1 0)
-		(unit 1)
-		(exclude_from_sim no)
-		(in_bom yes)
-		(on_board yes)
-		(dnp no)
-		(fields_autoplaced yes)
-		(property "Reference" "#PWR036"
-			(at 240.03 41.91 0)
-			(effects
-				(font
-					(size 1.27 1.27)
-				)
-				(hide yes)
-			)
-		)
-		(property "Value" "+5V"
-			(at 240.03 33.02 0)
-			(effects
-				(font
-					(size 1.27 1.27)
-				)
-			)
-		)
-		(property "Footprint" ""
-			(at 240.03 38.1 0)
-			(effects
-				(font
-					(size 1.27 1.27)
-				)
-				(hide yes)
-			)
-		)
-		(property "Datasheet" ""
-			(at 240.03 38.1 0)
-			(effects
-				(font
-					(size 1.27 1.27)
-				)
-				(hide yes)
-			)
-		)
-		(property "Description" "Power symbol creates a global label with name \"+5V\""
-			(at 240.03 38.1 0)
-			(effects
-				(font
-					(size 1.27 1.27)
-				)
-				(hide yes)
-			)
-		)
-		(pin "1"
-		)
-		(instances
-			(project ""
-				(path "/caf1b85f-a91d-4c85-9df1-65f9ebc85027/98cbb8f8-8dc6-43c0-8573-4a0e6318dc31"
-					(reference "#PWR036")
-					(unit 1)
-				)
-			)
-		)
-	)
-	(symbol
 		(lib_id "Device:C")
 		(at 140.97 111.76 0)
@@
 			)
 		)
-		(property "Value" "6u8"
+		(property "Value" "10u"
 			(at 153.67 45.7199 0)
 			(effects
@@
 	)
 	(symbol
+		(lib_id "power:+3.3V")
+		(at 240.03 36.83 0)
+		(unit 1)
+		(exclude_from_sim no)
+		(in_bom yes)
+		(on_board yes)
+		(dnp no)
+		(fields_autoplaced yes)
+		(property "Reference" "#PWR036"
+			(at 240.03 40.64 0)
+			(effects
+				(font
+					(size 1.27 1.27)
+				)
+				(hide yes)
+			)
+		)
+		(property "Value" "+3.3V"
+			(at 240.03 31.75 0)
+			(effects
+				(font
+					(size 1.27 1.27)
+				)
+			)
+		)
+		(property "Footprint" ""
+			(at 240.03 36.83 0)
+			(effects
+				(font
+					(size 1.27 1.27)
+				)
+				(hide yes)
+			)
+		)
+		(property "Datasheet" ""
+			(at 240.03 36.83 0)
+			(effects
+				(font
+					(size 1.27 1.27)
+				)
+				(hide yes)
+			)
+		)
+		(property "Description" "Power symbol creates a global label with name \"+3.3V\""
+			(at 240.03 36.83 0)
+			(effects
+				(font
+					(size 1.27 1.27)
+				)
+				(hide yes)
+			)
+		)
+		(pin "1"
+		)
+		(instances
+			(project ""
+				(path "/caf1b85f-a91d-4c85-9df1-65f9ebc85027/98cbb8f8-8dc6-43c0-8573-4a0e6318dc31"
+					(reference "#PWR036")
+					(unit 1)
+				)
+			)
+		)
+	)
+	(symbol
 		(lib_id "power:GND")
 		(at 223.52 123.19 0)
@@
 			)
 		)
-		(property "Value" "1k"
+		(property "Value" "220"
 			(at 107.95 83.8199 0)
 			(effects
@@
 			)
 		)
-		(property "Value" "15u"
+		(property "Value" "10u"
 			(at 201.93 34.29 90)
 			(effects
@@
 			)
 		)
-		(property "Value" "LED"
+		(property "Value" "LED_GREEN"
 			(at 93.0275 69.85 0)
 			(effects
@@
 			)
 		)
-		(property "Value" "13k7"
+		(property "Value" "22k"
 			(at 220.98 55.8799 0)
 			(effects

Commit message: Add lock file for ALBERT_FLIGHTCOMPUTER PCB design
Parts:
- removed C20, C22: 10u, symbol Device:C
- removed C44: 2n2, symbol Device:C
- removed IC2: TPS621351RGXR, TPS621361RGXT, symbol TPS621351RGXR:TPS621351RGXR
- removed J3: XT60-M, XT60-M:AMASS_XT60-M, symbol New_Library_1:XT60-M
- removed L2: 1u, symbol Device:L_Iron_Small
- removed R7: 1M1, symbol Device:R
- removed R8, R9: 100k, symbol Device:R
- added H1, H2, H3, H4: MountingHole, MountingHole:MountingHole_3.2mm_M3, symbol Mechanical:MountingHole
- added J17: XT60-M, XT60-M:AMASS_XT60-M, symbol New_Library_1:XT60-M
- added JP3: SolderJumper_2_Open, Jumper:SolderJumper-2_P1.3mm_Open_RoundedPad1.0x1.5mm, symbol Jumper:SolderJumper_2_Open
- added TP2: TestPoint 3V3, TestPoint:TestPoint_Pad_D2.5mm, symbol Connector:TestPoint
- C41: renamed from C13; footprint (none) -> Capacitor_SMD:C_0805_2012Metric
- C45: renamed from C14; footprint (none) -> Capacitor_SMD:C_0805_2012Metric
- C46: renamed from C19; footprint (none) -> CL32A106KBJNNNE:CAPC3225X270N
- C50: renamed from C21; footprint (none) -> Capacitor_SMD:C_0402_1005Metric
- C58: renamed from C23; footprint (none) -> GRM32ER61C476KE15L:CAPC3225X270N
- C59: renamed from C24; footprint (none) -> Capacitor_SMD:C_0402_1005Metric
- D7: renamed from D1; footprint (none) -> LED_SMD:LED_0603_1608Metric
- L2: renamed from L1; footprint (none) -> XAL5050-822MEC:XAL5050822MEC
- R38: renamed from R6; footprint (none) -> Resistor_SMD:R_2512_6332Metric
- R42: renamed from R2; footprint (none) -> Resistor_SMD:R_0402_1005Metric
- R44: renamed from R10; footprint (none) -> Resistor_SMD:R_0402_1005Metric
- R45: renamed from R11; footprint (none) -> Resistor_SMD:R_0402_1005Metric
- renumbered U2 to U4, U6 to U5, U7 to U6
Connections:
- net +3.3V: now also JP3.2 (B); no longer C58.1, L2.2, R44.1
- net GND: now also J17.N (NEG)
- net IN+: now also J17.P (POS)
- new net: C58.1, JP3.1 (A), L2.2, R44.1, TP2.1
Other:
- note added: "Buck Converter 1 12V/3V3"
- note added: "Mounting Holes"
- note added: "POWER FLAGS"
- note removed: "Buck Converter DOS 12V/8,4V"
- note removed: "Buck Converter UNO 12V/3V3"
- note removed: "C19 - ceramic C21 - ceramic pay attention to the max voltage ratings of the caps"
- company: (none) -> ALBERT AEROSPACE
- moved on the sheet: C41, C45, C46, C50, C58, C59, D7, L2, R38, R42, R44, R45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

Commit message: update pcb
Other:
- moved on the sheet: H1, H2, H3, H4
Changed lines of the file:
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@@
 	)
 	(rectangle
-		(start 17.78 160.02)
-		(end 63.5 179.07)
+		(start 19.05 90.17)
+		(end 64.77 109.22)
 		(stroke
 			(width 0)
@@
 	)
 	(rectangle
-		(start 87.63 160.02)
-		(end 116.84 186.69)
+		(start 88.9 90.17)
+		(end 118.11 116.84)
 		(stroke
 			(width 0)
@@
 	(text "Mounting Holes"
 		(exclude_from_sim no)
-		(at 94.742 188.722 0)
+		(at 96.012 118.872 0)
 		(effects
 			(font
@@
 	(text "POWER FLAGS"
 		(exclude_from_sim no)
-		(at 24.13 180.594 0)
+		(at 25.4 110.744 0)
 		(effects
 			(font
@@
 	(wire
 		(pts
-			(xy 54.61 167.64) (xy 54.61 171.45)
+			(xy 55.88 97.79) (xy 55.88 101.6)
 		)
 		(stroke
@@
 	(wire
 		(pts
-			(xy 24.13 167.64) (xy 24.13 171.45)
+			(xy 25.4 97.79) (xy 25.4 101.6)
 		)
 		(stroke
@@
 	(symbol
 		(lib_id "Mechanical:MountingHole")
-		(at 95.25 180.34 0)
+		(at 96.52 110.49 0)
 		(unit 1)
 		(exclude_from_sim yes)
@@
 		(fields_autoplaced yes)
 		(property "Reference" "H4"
-			(at 97.79 179.0699 0)
+			(at 99.06 109.2199 0)
 			(effects
 				(font
@@
 		)
 		(property "Value" "MountingHole"
-			(at 97.79 181.6099 0)
+			(at 99.06 111.7599 0)
 			(effects
 				(font
@@
 		)
 		(property "Footprint" "MountingHole:MountingHole_3.2mm_M3"
-			(at 95.25 180.34 0)
+			(at 96.52 110.49 0)
 			(effects
 				(font
@@
 		)
 		(property "Datasheet" "~"
-			(at 95.25 180.34 0)
+			(at 96.52 110.49 0)
 			(effects
 				(font
@@
 		)
 		(property "Description" "Mounting Hole without connection"
-			(at 95.25 180.34 0)
+			(at 96.52 110.49 0)
 			(effects
 				(font
@@
 	(symbol
 		(lib_id "Mechanical:MountingHole")
-		(at 95.25 170.18 0)
+		(at 96.52 100.33 0)
 		(unit 1)
 		(exclude_from_sim yes)
@@
 		(fields_autoplaced yes)
 		(property "Reference" "H2"
-			(at 97.79 168.9099 0)
+			(at 99.06 99.0599 0)
 			(effects
 				(font
@@
 		)
 		(property "Value" "MountingHole"
-			(at 97.79 171.4499 0)
+			(at 99.06 101.5999 0)
 			(effects
 				(font
@@
 		)
 		(property "Footprint" "MountingHole:MountingHole_3.2mm_M3"
-			(at 95.25 170.18 0)
+			(at 96.52 100.33 0)
 			(effects
 				(font
@@
 		)
 		(property "Datasheet" "~"
-			(at 95.25 170.18 0)
+			(at 96.52 100.33 0)
 			(effects
 				(font
@@
 		)
 		(property "Description" "Mounting Hole without connection"
-			(at 95.25 170.18 0)
+			(at 96.52 100.33 0)
 			(effects
 				(font
@@
 	(symbol
 		(lib_id "power:PWR_FLAG")
-		(at 24.13 171.45 180)
+		(at 25.4 101.6 180)
 		(unit 1)
 		(exclude_from_sim no)
@@
 		(fields_autoplaced yes)
 		(property "Reference" "#FLG03"
-			(at 24.13 173.355 0)
+			(at 25.4 103.505 0)
 			(effects
 				(font
@@
 		)
 		(property "Value" "PWR_FLAG"
-			(at 24.13 176.53 0)
+			(at 25.4 106.68 0)
 			(effects
 				(font
@@
 		)
 		(property "Footprint" ""
-			(at 24.13 171.45 0)
+			(at 25.4 101.6 0)
 			(effects
 				(font
@@
 		)
 		(property "Datasheet" "~"
-			(at 24.13 171.45 0)
+			(at 25.4 101.6 0)
 			(effects
 				(font
@@
 		)
 		(property "Description" "Special symbol for telling ERC where power comes from"
-			(at 24.13 171.45 0)
+			(at 25.4 101.6 0)
 			(effects
 				(font
@@
 	(symbol
 		(lib_id "power:VBUS")
-		(at 24.13 167.64 0)
+		(at 25.4 97.79 0)
 		(unit 1)
 		(exclude_from_sim no)
@@
 		(fields_autoplaced yes)
 		(property "Reference" "#PWR098"
-			(at 24.13 171.45 0)
+			(at 25.4 101.6 0)
 			(effects
 				(font
@@
 		)
 		(property "Value" "VBAT"
-			(at 24.13 162.56 0)
+			(at 25.4 92.71 0)
 			(effects
 				(font
@@
 		)
 		(property "Footprint" ""
-			(at 24.13 167.64 0)
+			(at 25.4 97.79 0)
 			(effects
 				(font
@@
 		)
 		(property "Datasheet" ""
-			(at 24.13 167.64 0)
+			(at 25.4 97.79 0)
 			(effects
 				(font
@@
 		)
 		(property "Description" "Power symbol creates a global label with name \"VBUS\""
-			(at 24.13 167.64 0)
+			(at 25.4 97.79 0)
 			(effects
 				(font
@@
 	(symbol
 		(lib_id "Mechanical:MountingHole")
-		(at 95.25 165.1 0)
+		(at 96.52 95.25 0)
 		(unit 1)
 		(exclude_from_sim yes)
@@
 		(fields_autoplaced yes)
 		(property "Reference" "H1"
-			(at 97.79 163.8299 0)
+			(at 99.06 93.9799 0)
 			(effects
 				(font
@@
 		)
 		(property "Value" "MountingHole"
-			(at 97.79 166.3699 0)
+			(at 99.06 96.5199 0)
 			(effects
 				(font
@@
 		)
 		(property "Footprint" "MountingHole:MountingHole_3.2mm_M3"
-			(at 95.25 165.1 0)
+			(at 96.52 95.25 0)
 			(effects
 				(font
@@
 		)
 		(property "Datasheet" "~"
-			(at 95.25 165.1 0)
+			(at 96.52 95.25 0)
 			(effects
 				(font
@@
 		)
 		(property "Description" "Mounting Hole without connection"
-			(at 95.25 165.1 0)
+			(at 96.52 95.25 0)
 			(effects
 				(font
@@
 	(symbol
 		(lib_id "power:+5V")
-		(at 54.61 167.64 0)
+		(at 55.88 97.79 0)
 		(unit 1)
 		(exclude_from_sim no)
@@
 		(fields_autoplaced yes)
 		(property "Reference" "#PWR0100"
-			(at 54.61 171.45 0)
+			(at 55.88 101.6 0)
 			(effects
 				(font
@@
 		)
 		(property "Value" "+5V"
-			(at 54.61 162.56 0)
+			(at 55.88 92.71 0)
 			(effects
 				(font
@@
 		)
 		(property "Footprint" ""
-			(at 54.61 167.64 0)
+			(at 55.88 97.79 0)
 			(effects
 				(font
@@
 		)
 		(property "Datasheet" ""
-			(at 54.61 167.64 0)
+			(at 55.88 97.79 0)
 			(effects
 				(font
@@
 		)
 		(property "Description" "Power symbol creates a global label with name \"+5V\""
-			(at 54.61 167.64 0)
+			(at 55.88 97.79 0)
 			(effects
 				(font
@@
 	(symbol
 		(lib_id "Mechanical:MountingHole")
-		(at 95.25 175.26 0)
+		(at 96.52 105.41 0)
 		(unit 1)
 		(exclude_from_sim yes)
@@
 		(fields_autoplaced yes)
 		(property "Reference" "H3"
-			(at 97.79 173.9899 0)
+			(at 99.06 104.1399 0)
 			(effects
 				(font
@@
 		)
 		(property "Value" "MountingHole"
-			(at 97.79 176.5299 0)
+			(at 99.06 106.6799 0)
 			(effects
 				(font
@@
 		)
 		(property "Footprint" "MountingHole:MountingHole_3.2mm_M3"
-			(at 95.25 175.26 0)
+			(at 96.52 105.41 0)
 			(effects
 				(font
@@
 		)
 		(property "Datasheet" "~"
-			(at 95.25 175.26 0)
+			(at 96.52 105.41 0)
 			(effects
 				(font
@@
 		)
 		(property "Description" "Mounting Hole without connection"
-			(at 95.25 175.26 0)
+			(at 96.52 105.41 0)
 			(effects
 				(font
@@
 	(symbol
 		(lib_id "power:PWR_FLAG")
-		(at 54.61 171.45 180)
+		(at 55.88 101.6 180)
 		(unit 1)
 		(exclude_from_sim no)
@@
 		(fields_autoplaced yes)
 		(property "Reference" "#FLG05"
-			(at 54.61 173.355 0)
+			(at 55.88 103.505 0)
 			(effects
 				(font
@@
 		)
 		(property "Value" "PWR_FLAG"
-			(at 54.61 176.53 0)
+			(at 55.88 106.68 0)
 			(effects
 				(font
@@
 		)
 		(property "Footprint" ""
-			(at 54.61 171.45 0)
+			(at 55.88 101.6 0)
 			(effects
 				(font
@@
 		)
 		(property "Datasheet" "~"
-			(at 54.61 171.45 0)
+			(at 55.88 101.6 0)
 			(effects
 				(font
@@
 		)
 		(property "Description" "Special symbol for telling ERC where power comes from"
-			(at 54.61 171.45 0)
+			(at 55.88 101.6 0)
 			(effects
 				(font

Commit message: Add production files and update project lock file
- Added new production IT1 zip file for ALBERT_FLIGHTCOMPUTER.
- Removed obsolete test zip file from production directory.
- Created a lock file for the KiCad schematic with user and hostname information.
Parts:
- C41, C45: LCSC (none) -> C45783
- C46: LCSC (none) -> C380537
- C50, C59: LCSC (none) -> C1525
- C58: LCSC (none) -> C77101
- J17: LCSC (none) -> C98733
- JP3, TP2: now left out of the parts list
- L2: LCSC (none) -> C5309356
- R38: LCSC (none) -> C316229
- R42: LCSC (none) -> C25091
- R44: LCSC (none) -> C25741
- R45: LCSC (none) -> C25768
- U4: LCSC (none) -> C6186
- U5: LCSC (none) -> C168839
- U6: LCSC (none) -> C87469
Other:
- note removed: "Tantalum"
