File: 3_Flight_Computer/PCB/ALBERT_FLIGHTCOMPUTER/Power.kicad_sch (KiCad schematic)
At the start: 22 parts, among them J17 XT60-M, U4 AMS1117-3.3, U5 TPS54308, U6 INA219AxDCN

Commit message: Quid pro quo; bitch ich kriege einen ständer; bald steht der benz da; sunshine sunshine reggae; bakerman bada bada bada dada is baking bread; subaweya alaboya combagaweja
Connections:
- net PWR LED Kathode: no longer names the net of D7.1 (K), R42.1
Other:
- note added: "Buck Converter 8V/3V3"
- note removed: "Buck Converter 1 12V/3V3"
Changed lines of the file:
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@@
 		)
 	)
-	(text "Buck Converter 1 12V/3V3\n"
+	(text "Buck Converter 8V/3V3\n"
 		(exclude_from_sim no)
 		(at 151.13 67.31 0)
@@
 			(width 0)
 			(type default)
-		)
-	)
-	(label "PWR LED Kathode"
-		(at 101.6 64.77 0)
-		(effects
-			(font
-				(size 0.8 0.8)
-			)
-			(justify left bottom)
 		)
 	)
@@
 					(size 1.27 1.27)
 				)
-			)
-		)
+				(hide yes)
+			)
+		)

Commit message: Die EU ruft die Renaissance der Atomkraft aus – und Österreich schreit: "Schleich di!"
Other:
- company: ALBERT AEROSPACE -> ALBERT AERO
Changed lines of the file:
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@@
 		(date "2025-11-10")
 		(rev "0.1")
-		(company "ALBERT AEROSPACE")
+		(company "ALBERT AERO")
 	)
 	(rectangle
