File: 3_Flight_Computer/PCB/Neuer Ordner/untitled.kicad_sch (KiCad schematic)
At the start: 15 parts, among them J18 5-1814400-2, J19 5-1814400-2, U7 RFM95W-868S2, U8 ZOE-M8Q, Y3 32.768kHz

Commit message: hallo der papa is da
Parts:
- removed C60, C62: 100n, Capacitor_SMD:C_0402_1005Metric, symbol Device:C
- removed JP1: SolderJumper_2_Open, Jumper:SolderJumper-2_P1.3mm_Open_RoundedPad1.0x1.5mm, symbol Jumper:SolderJumper_2_Open
- removed Y3: 32.768kHz, Crystal:Crystal_SMD_MicroCrystal_CC7V-T1A-2Pin_3.2x1.5mm, symbol Device:Crystal
- added C50, C53: 100n, symbol Device:C
- added JP1: SolderJumper_3_Open, symbol Jumper:SolderJumper_3_Open
- added Y3: CM7V-T1A-32.768KHZ-6PF-20PPM-TA-QC, CM7V32768TBQA020, symbol CM7V-T1A-32_768KHZ-6PF-20PPM-T:CM7V-T1A-32.768KHZ-6PF-20PPM-TA-QC
- C51: renamed from C61; footprint CL21A475KOFNNNE:CAPC2012X135N -> (none); LCSC C1746 -> (none)
- C52: renamed from C63; footprint NFM18PC:NFM18PC474R0J3D -> NFM18PC474R0J3D; LCSC C478452 -> (none)
- D8: LCSC C233388 -> (none)
- FB5: footprint BLM15HD102SN1D:NFZ15SG152SN10B -> NFZ15SG152SN10B; LCSC C21516 -> (none)
- J13: renamed from J19; footprint 5-1814400-2:518144002 -> 518144002; LCSC C3174972 -> (none)
- J14: renamed from J18; footprint 5-1814400-2:518144002 -> 518144002; LCSC C3174972 -> (none)
- L3: footprint LQM21PN1R0MC0D:LQM21PN1R0MC0D -> LQM21PN1R0MC0D; LCSC C113100 -> (none)
- R43: renamed from R47; footprint Resistor_SMD:R_0402_1005Metric -> (none); LCSC C25077 -> (none)
- R44: renamed from R46; footprint Resistor_SMD:R_0402_1005Metric -> (none); LCSC C25744 -> (none)
- U1: renamed from U8; LCSC C7398634 -> (none)
- U8: renamed from U7; now in the parts list
Connections:
- net +3.3V: now also C50.1, C53.1, JP1.3 (B)
- net GND: now also U1.F3 (SQI_D3), C50.2, C53.2, JP1.1 (A)
- net at U1.C4 (~{SAFEBOOT}): now also JP1.2 (C)
- net GPS_INT: now reaches U1.G4 (PIO13/EXTINT)
- net at U1.J7 (RTC_I): now also Y3.2
- net at U1.J8 (RTC_O): now also Y3.1
- net SPI2_DIO0_MPU: no longer names the net of U8.14 (DIO0)
- net SPI2_DIO2_MPU: no longer names the net of U8.16 (DIO2)
- net SPI2_MOSI_MPU renamed SPI3_MOSI_NAV
- no-connect marks 12 -> 5
Other:
- note removed: "LORA Module"
- company: ALBERT AEROSPACE -> (none)
- title: GPS & LORA -> RF
- moved on the sheet: C51, C52, D8, FB5, J13, J14, L3, R43, R44, U1, U8
